Commit message: feat(description): 组装warehouse_robot（UR5 装上AGV + vacuum gripper + 摄像头)

File: robot_description/urdf/ur5/ur5.urdf.xacro (robot description, xacro)
@@ -2,20 +2,19 @@
 <robot xmlns:xacro="http://www.ros.org/wiki/xacro" name="ur5">
     <xacro:include filename="$(find robot_description)/urdf/ur5/ur5_macro.xacro"/>
-    <xacro:macro name="ur5_robot" params="prefix parent *origin">
-        <joint name="${prefix}base_mount" type="fixed">
-            <xacro:insert_block name="origin"/>
-            <parent link="${parent}"/>
-            <child link="${prefix}base_link"/>
-        </joint>
+    <xacro:macro name="ur5_robot" params="prefix parent">
         <xacro:ur_robot
-            prefix="${prefix}"
+            name="ur5"
+            tf_prefix="${prefix}"
+            parent="${parent}"
             joint_limits_parameters_file="$(find robot_description)/urdf/ur5/joint_limits.yaml"
             kinematics_parameters_file="$(find robot_description)/urdf/ur5/default_kinematics.yaml"
             physical_parameters_file="$(find robot_description)/urdf/ur5/physical_parameters.yaml"
-            visual_parameters_file="$(find robot_description)/urdf/ut5/visual_parameters.yaml"
-            transmission_hw_interface="hardware_interface/PositionJointInterface"
+            visual_parameters_file="$(find robot_description)/urdf/ur5/visual_parameters.yaml"
+            generate_ros2_control_tag="false"
             safety_limits="false"
             safety_pos_margin="0.15"
-            safety_k_position="20"/>
+            safety_k_position="20">
+            <origin xyz="0 0 0" rpy="0 0 0"/>
+        </xacro:ur_robot>
     </xacro:macro>
 </robot>
