Commit message: feat: 3个ArUco箱子模型 + camera plugin + rviz marker 可视化

File: robot_description/ros2_control/ur5_sim.ros2_control.xacro (robot description, xacro)
@@ -6,6 +6,7 @@
                 <plugin>gazebo_ros2_control/GazeboSystem</plugin>
             </hardware>
-            <xacro:macro name="ur5_joint" params="name">
+            <xacro:macro name="ur5_joint" params="name init_pos:=0.0">
                 <joint name="${prefix}${name}">
+                    <param name="initial_position">${init_pos}</param>
                     <command_interface name="position"/>
                     <command_interface name="velocity"/>
@@ -15,10 +16,10 @@
                 </joint>
             </xacro:macro>
-            <xacro:ur5_joint name="shoulder_pan_joint"/>
-            <xacro:ur5_joint name="shoulder_lift_joint"/>
-            <xacro:ur5_joint name="elbow_joint"/>
-            <xacro:ur5_joint name="wrist_1_joint"/>
-            <xacro:ur5_joint name="wrist_2_joint"/>
-            <xacro:ur5_joint name="wrist_3_joint"/>
+            <xacro:ur5_joint name="shoulder_pan_joint"  init_pos="0.0"/>
+            <xacro:ur5_joint name="shoulder_lift_joint" init_pos="-1.5708"/>
+            <xacro:ur5_joint name="elbow_joint"         init_pos="1.5708"/>
+            <xacro:ur5_joint name="wrist_1_joint"       init_pos="-1.5708"/>
+            <xacro:ur5_joint name="wrist_2_joint"       init_pos="-1.5708"/>
+            <xacro:ur5_joint name="wrist_3_joint"       init_pos="0.0"/>
         </ros2_control>
     </xacro:macro>

File: robot_description/urdf/warehouse_agv/warehouse_agv.urdf.xacro (robot description, xacro)
@@ -31,5 +31,6 @@
             </collision>
             <inertial>
-                <origin xyz="0 0 ${base_height/2}" rpy="0 0 0"/>
+                <!-- Lower the CoM to just above the wheel axle to keep the AGV stable in Gazebo -->
+                <origin xyz="0 0 0.02" rpy="0 0 0"/>
                 <mass value="${base_mass}"/>
                 <xacro:box_inertia m="${base_mass}" x="${base_length}" y="${base_width}" z="${base_height}"/>
@@ -87,15 +88,17 @@
         <gazebo reference="${prefix}left_wheel_link">
             <mu1>1.0</mu1><mu2>1.0</mu2>
-            <kp>1e7</kp><kd>1.0</kd>
+            <kp>1e6</kp><kd>10.0</kd>
         </gazebo>
         <gazebo reference="${prefix}right_wheel_link">
             <mu1>1.0</mu1><mu2>1.0</mu2>
-            <kp>1e7</kp><kd>1.0</kd>
+            <kp>1e6</kp><kd>10.0</kd>
         </gazebo>
         <gazebo reference="${prefix}front_caster_link">
-            <mu1>0.0</mu1><mu2>0.0</mu2>
+            <mu1>0.2</mu1><mu2>0.2</mu2>
+            <kp>1e6</kp><kd>10.0</kd>
         </gazebo>
         <gazebo reference="${prefix}back_caster_link">
-            <mu1>0.0</mu1><mu2>0.0</mu2>
+            <mu1>0.2</mu1><mu2>0.2</mu2>
+            <kp>1e6</kp><kd>10.0</kd>
         </gazebo>
     </xacro:macro>

File: robot_description/urdf/warehouse_robot.urdf.xacro (robot description, xacro)
@@ -36,4 +36,17 @@
     <xacro:ur5_ros2_control_sim prefix="ur5_"/>
     <xacro:agv_ros2_control_sim prefix=""/>
+    <gazebo reference="camera_link">
+        <sensor type="camera" name="camera">
+            <update_rate>15.0</update_rate>
+            <camera>
+                <horizontal_fov>1.0472</horizontal_fov>
+                <image><width>640</width><height>480</height><format>R8G8B8</format></image>
+                <clip><near>0.05</near><far>10</far></clip>
+            </camera>
+            <plugin name="camera_driver" filename="libgazebo_ros_camera.so">
+                <frame_name>camera_color_optical_frame</frame_name>
+            </plugin>
+        </sensor>
+    </gazebo>
     <gazebo>
         <plugin filename="libgazebo_ros2_control.so" name="gazebo_ros2_control">
