Commit message: feat(sim): 调整AGV摩擦系数与UR5阻尼; 新增 warehouse.world 占位

File: robot_description/urdf/warehouse_agv/warehouse_agv.urdf.xacro (robot description, xacro)
@@ -41,5 +41,5 @@
             <parent link="${prefix}base_link"/>
             <child link="${prefix}arm_mount_link"/>
-            <orgin xyz="-0.05 0 ${base_height + 0.05}" rpy="0 0 0"/>
+            <origin xyz="-0.05 0 ${base_height + 0.05}" rpy="0 0 0"/>
         </joint>
         <!-- diff drive wheels -->
@@ -85,4 +85,18 @@
         <xacro:caster name="front" x_offset="0.25"/>
         <xacro:caster name="back" x_offset="-0.25"/>
+        <gazebo reference="${prefix}left_wheel_link">
+            <mu1>1.0</mu1><mu2>1.0</mu2>
+            <kp>1e7</kp><kd>1.0</kd>
+        </gazebo>
+        <gazebo reference="${prefix}right_wheel_link">
+            <mu1>1.0</mu1><mu2>1.0</mu2>
+            <kp>1e7</kp><kd>1.0</kd>
+        </gazebo>
+        <gazebo reference="${prefix}front_caster_link">
+            <mu1>0.0</mu1><mu2>0.0</mu2>
+        </gazebo>
+        <gazebo reference="${prefix}back_caster_link">
+            <mu1>0.0</mu1><mu2>0.0</mu2>
+        </gazebo>
     </xacro:macro>
 </robot>

File: robot_description/urdf/warehouse_robot.urdf.xacro (robot description, xacro)
@@ -4,4 +4,5 @@
     <xacro:include filename="$(find robot_description)/urdf/ur5/ur5.urdf.xacro"/>
     <xacro:include filename="$(find robot_description)/urdf/grippers/vacuum_gripper.urdf.xacro"/>
+    <xacro:include filename="$(find robot_simulation)/gazebo/warehouse_robot.gazebo.xacro"/>
     <!-- Mobile base -->
     <xacro:warehouse_agv_robot prefix=""/>

Commit message: 修复AGV静止后退蠕动（驱动轮轴对齐合质心）

File: robot_description/urdf/warehouse_agv/warehouse_agv.urdf.xacro (robot description, xacro)
@@ -8,4 +8,5 @@
     <xacro:property name="wheel_width" value="0.04"/>
     <xacro:property name="wheel_separation" value="0.42"/>
+    <xacro:property name="wheel_x_offset" value="-0.017"/>  <!-- shift drive axle under combined base+UR5 CoM to stop idle creep -->
     <xacro:macro name="box_inertia" params="m x y z">
         <inertia ixx="${m*(y*y+z*z)/12.0}" ixy="0" ixz="0"
@@ -64,5 +65,5 @@
                 <parent link="${prefix}base_link"/>
                 <child link="${prefix}${side}_wheel_link"/>
-                <origin xyz="0 ${y_reflect * wheel_separation/2} 0" rpy="0 0 0"/>
+                <origin xyz="${wheel_x_offset} ${y_reflect * wheel_separation/2} 0" rpy="0 0 0"/>
                 <axis xyz="0 1 0"/>
             </joint>
@@ -88,16 +89,16 @@
         <gazebo reference="${prefix}left_wheel_link">
             <mu1>1.0</mu1><mu2>1.0</mu2>
-            <kp>1e6</kp><kd>10.0</kd>
+            <kp>1e7</kp><kd>1.0</kd>
         </gazebo>
         <gazebo reference="${prefix}right_wheel_link">
             <mu1>1.0</mu1><mu2>1.0</mu2>
-            <kp>1e6</kp><kd>10.0</kd>
+            <kp>1e7</kp><kd>1.0</kd>
         </gazebo>
         <gazebo reference="${prefix}front_caster_link">
-            <mu1>0.2</mu1><mu2>0.2</mu2>
+            <mu1>0.0</mu1><mu2>0.0</mu2>
             <kp>1e6</kp><kd>10.0</kd>
         </gazebo>
         <gazebo reference="${prefix}back_caster_link">
-            <mu1>0.2</mu1><mu2>0.2</mu2>
+            <mu1>0.0</mu1><mu2>0.0</mu2>
             <kp>1e6</kp><kd>10.0</kd>
         </gazebo>

Commit message: Fix/agv drift (#17)
修复AGV静止后退蠕动（驱动轮轴对齐合质心）

File: robot_description/urdf/warehouse_agv/warehouse_agv.urdf.xacro (robot description, xacro)
@@ -8,4 +8,5 @@
     <xacro:property name="wheel_width" value="0.04"/>
     <xacro:property name="wheel_separation" value="0.42"/>
+    <xacro:property name="wheel_x_offset" value="-0.017"/>  <!-- shift drive axle under combined base+UR5 CoM to stop idle creep -->
     <xacro:macro name="box_inertia" params="m x y z">
         <inertia ixx="${m*(y*y+z*z)/12.0}" ixy="0" ixz="0"
@@ -64,5 +65,5 @@
                 <parent link="${prefix}base_link"/>
                 <child link="${prefix}${side}_wheel_link"/>
-                <origin xyz="0 ${y_reflect * wheel_separation/2} 0" rpy="0 0 0"/>
+                <origin xyz="${wheel_x_offset} ${y_reflect * wheel_separation/2} 0" rpy="0 0 0"/>
                 <axis xyz="0 1 0"/>
             </joint>
@@ -95,9 +96,9 @@
         </gazebo>
         <gazebo reference="${prefix}front_caster_link">
-            <mu1>0.2</mu1><mu2>0.2</mu2>
+            <mu1>0.0</mu1><mu2>0.0</mu2>
             <kp>1e6</kp><kd>10.0</kd>
         </gazebo>
         <gazebo reference="${prefix}back_caster_link">
-            <mu1>0.2</mu1><mu2>0.2</mu2>
+            <mu1>0.0</mu1><mu2>0.0</mu2>
             <kp>1e6</kp><kd>10.0</kd>
         </gazebo>
