Commit message: feat(decision): auto_pick_node -- 感知subscriber 接 PickAndPlace action client

File: robot_control/moveit_config/ur5_warehouse_moveit_config/config/warehouse_robot.urdf.xacro (robot description, xacro)
@@ -3,5 +3,5 @@
     <xacro:arg name="initial_positions_file" default="initial_positions.yaml" />
     <!-- Import warehouse_robot urdf file -->
-    <xacro:include filename="$(find moveit_resources_panda_description)/urdf/warehouse_robot.urdf" />
+    <xacro:include filename="$(find robot_description)/urdf/warehouse_robot.urdf.xacro" />
     <!-- Import control_xacro -->
     <xacro:include filename="warehouse_robot.ros2_control.xacro" />

File: robot_description/urdf/grippers/vacuum_gripper.urdf.xacro (robot description, xacro)
@@ -1,5 +1,5 @@
 <?xml version="1.0"?>
 <robot xmlns:xacro="http://www.ros.org/wiki/xacro" name="vacuum_gripper">
-    <xacro:macro name="vacuum_gripper" params="prefix parent">
+    <xacro:macro name="vacuum_gripper" params="prefix parent gazebo_link">
         <link name="${prefix}vacuum_base_link">
             <visual>
@@ -22,6 +22,22 @@
             <origin xyz="0 0 0" rpy="0 0 0"/>
         </joint>
-        <!-- TCP - contact surface of suction cup, used by MoveIt as end-effector frame -->
-        <link name="${prefix}vacuum_tcp"/>
+        <gazebo reference="${prefix}vacuum_mount_joint">
+            <preserveFixedJoint>true</preserveFixedJoint>
+            <disableFixedJointLumping>true</disableFixedJointLumping>
+        </gazebo>
+        <!-- TCP - contact surface of suction cup, used by MoveIt. Gazebo's URDF
+             conversion merges fixed child links, so the vacuum plugin binds to
+             the nearest preserved Gazebo link and uses max_distance to reach it. -->
+        <link name="${prefix}vacuum_tcp">
+            <visual>
+                <origin xyz="0 0 0"/>
+                <geometry><cylinder radius="0.026" length="0.004"/></geometry>
+                <material name="suction_tip_blue"><color rgba="0.1 0.25 0.9 0.7"/></material>
+            </visual>
+            <inertial>
+                <mass value="0.005"/>
+                <inertia ixx="1e-6" iyy="1e-6" izz="1e-6" ixy="0" ixz="0" iyz="0"/>
+            </inertial>
+        </link>
         <joint name="${prefix}vacuum_tcp_joint" type="fixed">
             <parent link="${prefix}vacuum_base_link"/>
@@ -29,4 +45,25 @@
             <origin xyz="0 0 0.05" rpy="0 0 0"/>
         </joint>
+        <gazebo reference="${prefix}vacuum_tcp_joint">
+            <preserveFixedJoint>true</preserveFixedJoint>
+            <disableFixedJointLumping>true</disableFixedJointLumping>
+        </gazebo>
+        <gazebo>
+            <plugin name="${prefix}vacuum_gripper" filename="libgazebo_ros_vacuum_gripper.so">
+                <ros>
+                    <namespace>/vacuum_gripper</namespace>
+                </ros>
+                <link_name>${gazebo_link}</link_name>
+                <!-- The plugin checks distance from the vacuum link origin to
+                     object link origins. A 0.10 m box with TCP clearance plus
+                     small AGV/Gazebo base drift needs more than the box half
+                     height alone. Keep this below the neighboring box distance. -->
+                <max_distance>0.18</max_distance>
+                <fixed>warehouse_robot</fixed>
+                <fixed>ground_plane</fixed>
+                <fixed>sun</fixed>
+                <fixed>aruco_platform</fixed>
+            </plugin>
+        </gazebo>
     </xacro:macro>
 </robot>

File: robot_description/urdf/warehouse_agv/warehouse_agv.urdf.xacro (robot description, xacro)
@@ -67,4 +67,5 @@
                 <origin xyz="${wheel_x_offset} ${y_reflect * wheel_separation/2} 0" rpy="0 0 0"/>
                 <axis xyz="0 1 0"/>
+                <dynamics damping="1.0" friction="1.0"/>
             </joint>
         </xacro:macro>
@@ -88,18 +89,28 @@
         <xacro:caster name="back" x_offset="-0.25"/>
         <gazebo reference="${prefix}left_wheel_link">
-            <mu1>1.0</mu1><mu2>1.0</mu2>
-            <kp>1e6</kp><kd>10.0</kd>
+            <mu1>500.0</mu1><mu2>500.0</mu2>
+            <kp>1000000.0</kp><kd>10.0</kd>
+            <minDepth>0.001</minDepth>
+            <maxVel>0.1</maxVel>
+            <fdir1>1 0 0</fdir1>
         </gazebo>
         <gazebo reference="${prefix}right_wheel_link">
-            <mu1>1.0</mu1><mu2>1.0</mu2>
-            <kp>1e6</kp><kd>10.0</kd>
+            <mu1>500.0</mu1><mu2>500.0</mu2>
+            <kp>1000000.0</kp><kd>10.0</kd>
+            <minDepth>0.001</minDepth>
+            <maxVel>0.1</maxVel>
+            <fdir1>1 0 0</fdir1>
         </gazebo>
         <gazebo reference="${prefix}front_caster_link">
-            <mu1>0.0</mu1><mu2>0.0</mu2>
-            <kp>1e6</kp><kd>10.0</kd>
+            <mu1>0.1</mu1><mu2>0.1</mu2>
+            <kp>1000000.0</kp><kd>10.0</kd>
+            <minDepth>0.001</minDepth>
+            <maxVel>1.0</maxVel>
         </gazebo>
         <gazebo reference="${prefix}back_caster_link">
-            <mu1>0.0</mu1><mu2>0.0</mu2>
-            <kp>1e6</kp><kd>10.0</kd>
+            <mu1>0.1</mu1><mu2>0.1</mu2>
+            <kp>1000000.0</kp><kd>10.0</kd>
+            <minDepth>0.001</minDepth>
+            <maxVel>1.0</maxVel>
         </gazebo>
     </xacro:macro>

File: robot_description/urdf/warehouse_robot.urdf.xacro (robot description, xacro)
@@ -11,6 +11,8 @@
     <!-- UR5 mounted on arm_mount_link of AGV. z-offset already in arm_mount_joint. -->
     <xacro:ur5_robot prefix="ur5_" parent="arm_mount_link"/>
-    <!-- Vacuum gripper attached to UR5 tool0 -->
-    <xacro:vacuum_gripper prefix="" parent="ur5_tool0"/>
+    <!-- Vacuum gripper physical link attached directly to the stable Gazebo wrist link.
+         ur5_tool0 has the same transform as ur5_wrist_3_link in this URDF and remains
+         available as the MoveIt planning frame. -->
+    <xacro:vacuum_gripper prefix="" parent="ur5_wrist_3_link" gazebo_link="vacuum_tcp"/>
     <!-- Camera (Eye-to-Hand) fixed on AGV body, looking forward+down -->
     <link name="camera_link">
@@ -54,11 +56,3 @@
         </plugin>
     </gazebo>
-    <gazebo>
-        <plugin name="vacuum_gripper" filename="libgazebo_ros_vacuum_gripper.so">
-            <ros><namespace>/vacuum_gripper</namespace></ros>
-            <link_name>vacuum_base_link</link_name>
-            <fixed>base_link</fixed>
-            <max_distance>0.05</max_distance>
-        </plugin>
-    </gazebo>
 </robot>
