Commit message: feat(control): 成功实现连续3次detect-pick-place

File: robot_description/urdf/warehouse_robot.urdf.xacro (robot description, xacro)
@@ -27,5 +27,5 @@
         <parent link="base_link"/>
         <child link="camera_link"/>
-        <origin xyz="0.30 0 0.30" rpy="0 0.5236 0"/>    <!-- pitched 30 deg down -->
+        <origin xyz="0.30 0 0.30" rpy="0 0.7854 0"/>    <!-- pitched 30 deg down -->
     </joint>
     <!-- Optical frame - REP-103 convention (x right, y down, z forward) -->
@@ -43,5 +43,5 @@
             <camera>
                 <horizontal_fov>1.0472</horizontal_fov>
-                <image><width>640</width><height>480</height><format>R8G8B8</format></image>
+                <image><width>1280</width><height>720</height><format>R8G8B8</format></image>
                 <clip><near>0.05</near><far>10</far></clip>
             </camera>
